File: Receiver/ReceiverBoard/ReceiverBoard.kicad_sch (KiCad schematic)
At the start: 57 parts, among them IC1 SN74HCT245PWR, IC2 SN74HCT245PWR, J1 Left Header, J10 Output 5, J11 Output 6, J12 Output 7, J13 High Power, J14 Output 8, J15 Output 9, J16 Output 10, J17 Output 11, J18 Output 12, J19 Output 13, J2 Right Header, J20 Output 14, J21 Output 15, J22 J1B1211CCD, J3 Upper Middle Header, J4 Lower Middle Header, J5 Output 0, J6 Output 1, J7 Output 2, J8 Output 3, J9 Output 4, U0 Data, U1 Teensy4.1, U1 UCS2904, U2 UCS2904, U3 UCS2904

Commit message: Artnet is up and running!
Parts:
- removed D1, D2, D3: RGBWLed (x12), symbol Polis_Symbols:RGBWLed
- removed H2, H3, H4: MountingHole, MountingHole:MountingHole_3.2mm_M3, symbol Mechanical:MountingHole
- removed J13: High Power, Connector_AMASS:AMASS_XT30U-F_1x02_P5.0mm_Vertical, symbol Connector:Conn_01x02_Socket
- removed J3: Upper Middle Header, Connector_PinHeader_2.00mm:PinHeader_1x03_P2.00mm_Vertical, symbol Connector:Conn_01x03_Socket
- removed J4: Lower Middle Header, Connector_PinHeader_2.00mm:PinHeader_1x03_P2.00mm_Vertical, symbol Connector:Conn_01x03_Socket
- removed U0: Data, symbol Connector:Conn_01x03_Pin
- removed U1, U2, U3: UCS2904, symbol Polis_Symbols:UCS2904
- added C1: 1000u, Capacitor_THT:C_Radial_D16.0mm_H25.0mm_P7.50mm, symbol Device:C_Small
- added C4: 1u, Capacitor_SMD:C_0603_1608Metric_Pad1.08x0.95mm_HandSolder, symbol Device:C_Small
- added D1, D26: RED, LED_SMD:LED_1206_3216Metric_Pad1.42x1.75mm_HandSolder, symbol Device:LED
- added D10, D11, D12, D13, D14, D15, D16, D17, D18, D19, D2, D20, D21, D22, D23, D24, D25, D3, D4, D5, D6, D7, D8, D9: YELLOW, LED_SMD:LED_0603_1608Metric_Pad1.05x0.95mm_HandSolder, symbol Device:LED
- added H2, H3, H4: MountingHole, MountingHole:MountingHole_3.2mm_M3_Pad, symbol Mechanical:MountingHole_Pad
- added IC3: SN74HCT245PWR, SOP65P640X120-20N, symbol SN74HCT245PWR:SN74HCT245PWR
- added J13, J22, J23, J24, J25, J26, J27, J28: String, SHDR3W80P0X350_1X3_1250X725X940P, symbol 284514-3:284514-3
- added J3: Ethernet, Connector_PinHeader_2.00mm:PinHeader_2x03_P2.00mm_Vertical, symbol Connector_Generic:Conn_02x03_Odd_Even
- added J4: 1719312, 1719312:PHOENIX_1719312, symbol 1719312:1719312
- added R17, R18, R19, R20, R21, R22, R23, R24, R25: 100, Resistor_SMD:R_0402_1005Metric_Pad0.72x0.64mm_HandSolder, symbol Device:R_Small_US
- added R26, R27, R28, R29, R30, R31, R32, R33, R34, R35, R36, R37, R38, R39, R40, R41, R42, R43, R44, R45, R46, R47, R48, R49: 3k, Resistor_SMD:R_0603_1608Metric_Pad0.98x0.95mm_HandSolder, symbol Device:R_Small_US
- added R50: 3.2k, Resistor_SMD:R_1206_3216Metric_Pad1.30x1.75mm_HandSolder, symbol Device:R_Small_US
- C2: renamed from C1; value 1uF -> 1u; footprint Capacitor_SMD:C_1206_3216Metric -> Capacitor_SMD:C_0603_1608Metric_Pad1.08x0.95mm_HandSolder; LCSC Part # (none) -> C576859
- C3: renamed from C2; value 1uF -> 1u; footprint Capacitor_SMD:C_1206_3216Metric -> Capacitor_SMD:C_0603_1608Metric_Pad1.08x0.95mm_HandSolder; LCSC Part # (none) -> C576859
- C5: renamed from C3; value 0.1uF -> 100n; footprint Capacitor_SMD:C_1206_3216Metric -> Capacitor_SMD:C_0603_1608Metric_Pad1.08x0.95mm_HandSolder; LCSC Part # (none) -> C161854
- H1: footprint MountingHole:MountingHole_3.2mm_M3 -> MountingHole:MountingHole_3.2mm_M3_Pad; symbol Mechanical:MountingHole -> Mechanical:MountingHole_Pad; now not fitted
- IC1, IC2: footprint SN74HCT245PWR:SOP65P640X120-20N -> SOP65P640X120-20N; LCSC Part # (none) -> C6779
- J1, J2: LCSC Part # (none) -> C2883520
- J10: value Output 5 -> String; footprint 284514-3:SHDR3W80P0X350_1X3_1250X725X940P -> SHDR3W80P0X350_1X3_1250X725X940P; LCSC Part # (none) -> C7466034
- J11: value Output 6 -> String; footprint 284514-3:SHDR3W80P0X350_1X3_1250X725X940P -> SHDR3W80P0X350_1X3_1250X725X940P; LCSC Part # (none) -> C7466034
- J12: value Output 7 -> String; footprint 284514-3:SHDR3W80P0X350_1X3_1250X725X940P -> SHDR3W80P0X350_1X3_1250X725X940P; LCSC Part # (none) -> C7466034
- J14: value Output 8 -> String; footprint 284514-3:SHDR3W80P0X350_1X3_1250X725X940P -> SHDR3W80P0X350_1X3_1250X725X940P; LCSC Part # (none) -> C7466034
- J15: value Output 9 -> String; footprint 284514-3:SHDR3W80P0X350_1X3_1250X725X940P -> SHDR3W80P0X350_1X3_1250X725X940P; LCSC Part # (none) -> C7466034
- J16: value Output 10 -> String; footprint 284514-3:SHDR3W80P0X350_1X3_1250X725X940P -> SHDR3W80P0X350_1X3_1250X725X940P; LCSC Part # (none) -> C7466034
- J17: value Output 11 -> String; footprint 284514-3:SHDR3W80P0X350_1X3_1250X725X940P -> SHDR3W80P0X350_1X3_1250X725X940P; LCSC Part # (none) -> C7466034; Mates with 284506-3 -> (none)
- J18: value Output 12 -> String; footprint 284514-3:SHDR3W80P0X350_1X3_1250X725X940P -> SHDR3W80P0X350_1X3_1250X725X940P; LCSC Part # (none) -> C7466034
- J19: value Output 13 -> String; footprint 284514-3:SHDR3W80P0X350_1X3_1250X725X940P -> SHDR3W80P0X350_1X3_1250X725X940P; LCSC Part # (none) -> C7466034
- J20: value Output 14 -> String; footprint 284514-3:SHDR3W80P0X350_1X3_1250X725X940P -> SHDR3W80P0X350_1X3_1250X725X940P; LCSC Part # (none) -> C7466034
- J21: value Output 15 -> String; footprint 284514-3:SHDR3W80P0X350_1X3_1250X725X940P -> SHDR3W80P0X350_1X3_1250X725X940P; LCSC Part # (none) -> C7466034
- J30: renamed from J22; value J1B1211CCD -> RVB-ZZ-0004; footprint J1B1211CCD:J1B1211CCD -> :RJ45-TH_RVB-ZZ-0004; symbol J1B1211CCD:J1B1211CCD -> RVB-ZZ-0004:RVB-ZZ-0004; LCSC Part # (none) -> C363242
- J5: value Output 0 -> String; footprint 284514-3:SHDR3W80P0X350_1X3_1250X725X940P -> SHDR3W80P0X350_1X3_1250X725X940P; LCSC Part # (none) -> C7466034
- J6: value Output 1 -> String; footprint 284514-3:SHDR3W80P0X350_1X3_1250X725X940P -> SHDR3W80P0X350_1X3_1250X725X940P; LCSC Part # (none) -> C7466034
- J7: value Output 2 -> String; footprint 284514-3:SHDR3W80P0X350_1X3_1250X725X940P -> SHDR3W80P0X350_1X3_1250X725X940P; LCSC Part # (none) -> C7466034
- J8: value Output 3 -> String; footprint 284514-3:SHDR3W80P0X350_1X3_1250X725X940P -> SHDR3W80P0X350_1X3_1250X725X940P; LCSC Part # (none) -> C7466034; Mates with 284506-3 -> (none)
- J9: value Output 4 -> String; footprint 284514-3:SHDR3W80P0X350_1X3_1250X725X940P -> SHDR3W80P0X350_1X3_1250X725X940P; LCSC Part # (none) -> C7466034
- JP1: LCSC Part # (none) -> C3325137
- PS1: footprint KiCad:TSR12450E -> TSR12450E; now not fitted
- R1: value 100 -> 3.3k; footprint Resistor_SMD:R_1206_3216Metric -> Resistor_SMD:R_1206_3216Metric_Pad1.30x1.75mm_HandSolder; LCSC Part # (none) -> C2089480
- R10, R11, R12, R13, R14, R15, R2, R3, R4, R5, R6, R7, R9: footprint Resistor_SMD:R_1206_3216Metric -> Resistor_SMD:R_0402_1005Metric_Pad0.72x0.64mm_HandSolder; LCSC Part # (none) -> C144045
- R16, R8: value 100(x8) -> 100; footprint Resistor_SMD:R_1206_3216Metric -> Resistor_SMD:R_0402_1005Metric_Pad0.72x0.64mm_HandSolder; LCSC Part # (none) -> C144045
- U1: now not fitted; now left out of the parts list
Connections:
- net +24V: now also C1.1, D1.2 (A), J13.3, J22.3, J23.3, J24.3, J25.3, J26.3, J27.3, J28.3, J4.2
- net +5V: now also C4.2, D26.2 (A), IC3.1 (DIR), IC3.20 (VCC)
- net D1: now also IC1.9 (A8), J2.24 (Pin_24); no longer IC1.8 (A7), J1.5 (Pin_5)
- net D10: now also IC2.8 (A7), J2.12 (Pin_12); no longer IC2.7 (A6), J2.13 (Pin_13)
- net D10O: now also J14.2, R11.2, D11.2 (A); no longer J16.2, R14.2
- net D11: now also IC2.7 (A6), J2.11 (Pin_11); no longer IC2.6 (A5), J2.12 (Pin_12)
- net D11O: now also J15.2, R12.2, D12.2 (A); no longer J17.2, R13.2
- net D12: now also IC2.6 (A5), J2.10 (Pin_10); no longer IC2.5 (A4), J2.9 (Pin_9)
- net D12O: now also J16.2, R13.2, D13.2 (A); no longer J18.2, R12.2
- net D13: now also IC2.5 (A4), J2.9 (Pin_9); no longer IC2.4 (A3), J2.8 (Pin_8)
- net D13O: now also J17.2, R14.2, D14.2 (A); no longer J19.2, R11.2
- net D14: now also IC2.4 (A3), J2.8 (Pin_8); no longer IC2.3 (A2), J2.5 (Pin_5)
- net D14O: now also J18.2, R15.2, D15.2 (A); no longer J20.2, R10.2
- net D15: now also IC2.3 (A2), J2.7 (Pin_7); no longer IC2.2 (A1), J2.4 (Pin_4)
- net D15O: now also J19.2, R16.2, D16.2 (A); no longer J21.2, R9.2
- net D1O: now also J5.2, R2.1, D2.2 (A); no longer J6.2, R7.2
- net D2: now also IC1.8 (A7), J2.23 (Pin_23); no longer IC1.7 (A6), J1.6 (Pin_6)
- net D2O: now also J6.2, R3.2, D3.2 (A); no longer J7.2, R6.2
- net D3: now also IC1.7 (A6), J2.22 (Pin_22); no longer IC1.6 (A5), J1.7 (Pin_7)
- net D3O: now also J7.2, R4.2, D4.2 (A); no longer J8.2, R5.2
- net D4: now also IC1.6 (A5), J2.21 (Pin_21); no longer IC1.5 (A4), J1.8 (Pin_8)
- net D4O: now also J8.2, R5.2, D5.2 (A); no longer J9.2, R4.2
- net D5: now also IC1.5 (A4), J2.20 (Pin_20); no longer IC1.4 (A3), J1.9 (Pin_9)
- net D5O: now also J9.2, R6.2, D6.2 (A); no longer J10.2, R3.2
- net D6: now also IC1.4 (A3), J2.19 (Pin_19); no longer IC1.3 (A2), J1.10 (Pin_10)
- net D6O: now also J10.2, R7.2, D7.2 (A); no longer J11.2, R2.2
- net D7: now also IC1.3 (A2), J2.18 (Pin_18); no longer IC1.2 (A1), J1.11 (Pin_11)
- net D7O: now also J11.2, R8.2, D8.2 (A); no longer J12.2, R1.2
- net D8: now also IC1.2 (A1), J2.17 (Pin_17); no longer IC2.9 (A8), J2.21 (Pin_21)
- net D8O: now also J12.2, R9.2, D9.2 (A); no longer J14.2, R16.2
- net D9: now also IC2.9 (A8), J2.13 (Pin_13); no longer IC2.8 (A7), J2.20 (Pin_20)
- net D9O: now also R10.1, D10.2 (A), J13.2; no longer J15.2, R15.2
- net ELED: now also J30.L2 (LED1+), J3.4 (Pin_4); no longer J30.10 (GLED+)
- net GND: now also H1.1, J30.13 (EH), J30.L1 (LED1-), J30.R8 (GND), R1.2, C1.2, C4.1, H2.1, H3.1, H4.1, IC3.10 (GND), IC3.19 (~{OE}), J13.1, J22.1, J23.1, J24.1, J25.1, J26.1, J27.1, J28.1, J3.3 (Pin_3), J4.1, R26.2, R27.2, R28.2, R29.2, R30.2, R31.2, R32.2, R33.1, R34.2, R35.2, R36.2, R37.2, R38.2, R39.2, R40.2, R41.2, R42.2, R43.2, R44.2, R45.2, R46.2, R47.2, R48.2, R49.2, R50.2; no longer J30.8 (GND), J30.9 (GLED-)
- net RX+: now also J30.R4 (RD+), J3.6 (Pin_6); no longer J30.4 (RD+)
- net RX-: now also J30.R6 (RD-), J3.5 (Pin_5); no longer J30.6 (RD-)
- net TX+: now also J30.R1 (TD+), J3.1 (Pin_1); no longer J30.1 (TD+)
- net TX-: now also J30.R3 (TD-), J3.2 (Pin_2); no longer J30.3 (TD-)
- net at IC2.11 (B8): now also R10.2; no longer R16.1
- net at IC2.12 (B7): now also R11.1; no longer R15.1
- net at IC2.13 (B6): now also R12.1; no longer R14.1
- net at IC2.15 (B4): now also R14.1; no longer R12.1
- net at IC2.16 (B3): now also R15.1; no longer R11.1
- net at IC2.17 (B2): now also R16.1; no longer R10.1
- net at R9.1: now also IC1.18 (B1); no longer IC2.18 (B1)
- net at IC1.15 (B4): now also R6.1; no longer R4.1
- net D16: now reaches J2.6 (Pin_6)
- net D16: now also IC2.2 (A1)
- net at IC1.13 (B6): now also R4.1; no longer R6.1
- net D22: now reaches J1.2 (Pin_2)
- net D22: now also IC3.4 (A3)
- net D23: now reaches J1.3 (Pin_3)
- net D23: now also IC3.3 (A2)
- net at IC1.11 (B8): now also R2.2; no longer R8.1
- net at R7.1: now also IC1.16 (B3); no longer IC1.12 (B7)
- net at R3.1: now also IC1.12 (B7); no longer IC1.16 (B3)
- net at IC1.17 (B2): now also R8.1; no longer R2.1
- net at R1.1: now also D1.1 (K); no longer IC1.18 (B1)
- net D0 renamed D24
- net D24: now also IC3.2 (A1); no longer IC1.9 (A8)
- removed net D0O: J5.2, R8.2
- new net: D19.1 (K), R43.1
- new net: D25.1 (K), R49.1
- new net: D17.1 (K), R41.1
- new net: D5.1 (K), R29.1
- new net: IC2.18 (B1), R17.1
- new net: D7.1 (K), R31.1
- new net: IC3.12 (B7), R19.1
- new net: D8.1 (K), R32.1
- new net: D14.1 (K), R38.1
- new net: C5.1, J30.R2 (TCT), J30.R5 (RCT)
- new net: D22.1 (K), R46.1
- new net: D26.1 (K), R50.1
- new net: D20.1 (K), R44.1
- new net: IC3.14 (B5), R21.1
- new net: D10.1 (K), R34.1
- new net: IC3.18 (B1), R25.1
- new net: D4.1 (K), R28.1
- new net: D6.1 (K), R30.1
- new net: D3.1 (K), R27.1
- new net: IC3.17 (B2), R24.1
- new net: D11.1 (K), R35.1
- new net: D23.1 (K), R47.1
- new net: D21.1 (K), R45.1
- new net: D9.1 (K), R33.2
- new net: IC3.13 (B6), R20.1
- new net: D24.1 (K), R48.1
- new net: D18.1 (K), R42.1
- new net: D13.1 (K), R37.1
- new net: D16.1 (K), R40.1
- new net: IC3.11 (B8), R18.2
- new net: IC3.15 (B4), R22.1
- new net: IC3.16 (B3), R23.1
- new net: D2.1 (K), R26.1
- new net: D12.1 (K), R36.1
- new net: D15.1 (K), R39.1
- new net D16O: D17.2 (A), J20.2, R17.2
- new net D17: IC3.9 (A8), J1.9 (Pin_9)
- new net D17O: D18.2 (A), J21.2, R18.1
- new net D18: IC3.8 (A7), J1.8 (Pin_8)
- new net D18O: D19.2 (A), J22.2, R19.2
- new net D19: IC3.7 (A6), J1.7 (Pin_7)
- new net D19O: D20.2 (A), J23.2, R20.2
- new net D20: IC3.6 (A5), J1.6 (Pin_6)
- new net D20O: D21.2 (A), J24.2, R21.2
- new net D21: IC3.5 (A4), J1.5 (Pin_5)
- new net D21O: D22.2 (A), J25.2, R22.2
- new net D22O: D23.2 (A), J26.2, R23.2
- new net D23O: D24.2 (A), J27.2, R24.2
- new net D24O: D25.2 (A), J28.2, R25.2
- no-connect marks 0 -> 20
Other:
- note removed: "..."
- note removed: "24V"
- note removed: "Controller"
- note removed: "Custom Board 1"
- note removed: "Custom Board 2"
- note removed: "Custom Board N"
- note removed: "Data"
- note removed: "GND"
- moved on the sheet: C2, C3, C5, IC1, IC2, J5, JP1
