File: Lamp/LampBoardModule/LampBoardModule.kicad_pcb (KiCad board)
At the start: 2 copper layers, 80 x 40 mm, 78 parts, among them IC1 L7805ABD2T-TR, IC2 SN74LVC2T45DCUR, J1 Conn_01x03_Socket, J2 Conn_01x03_Socket, J3 284514-3, J4 DC-005-A250, Q1 CMN3406M, SW1 PEC11R, SW2 MT-0-102, U1 RP2040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

Commit message: boards are done
Parts:
- removed REF**: MountingHole_2.7mm_M2.5_DIN965_Pad, MountingHole:MountingHole_2.7mm_M2.5_DIN965_Pad
- added D13: GREEN, LED_SMD:LED_0603_1608Metric, F.Cu at (74.0, 114.9)
- added G***: LOGO, Polis_Footprints:polis_logo_10x10, F.Cu at (65.2, 121.6)
- added H1: MountingHole_Pad, MountingHole:MountingHole_2.7mm_M2.5_DIN965_Pad, F.Cu at (48.0, 80.8)
- added H2: MountingHole_Pad, MountingHole:MountingHole_2.7mm_M2.5_DIN965_Pad, F.Cu at (48.0, 128.8)
- added H3: MountingHole_Pad, MountingHole:MountingHole_2.7mm_M2.5_DIN965_Pad, F.Cu at (121.0, 128.8)
- added H4: MountingHole_Pad, MountingHole:MountingHole_2.7mm_M2.5_DIN965_Pad, F.Cu at (121.0, 80.8)
- added R27: 330, Resistor_SMD:R_0603_1608Metric, F.Cu at (70.5, 114.9)
- added R28: 330, Resistor_SMD:R_0603_1608Metric, F.Cu at (72.3, 109.5)
- added R29: 10K, Resistor_SMD:R_0603_1608Metric, F.Cu at (71.8, 93.0)
- added R30: 1K, Resistor_SMD:R_0402_1005Metric, F.Cu at (54.7, 80.6)
- added R31: 1K, Resistor_SMD:R_0402_1005Metric, F.Cu at (53.4, 80.6)
- C1, C10, C11: footprint Capacitor_SMD:C_0603_1608Metric -> Capacitor_SMD:C_0402_1005Metric
- C12, C14, C16, C17, C18, C19, C20, C21, C22: value 100nF -> 100n
- C13, C15: value 1uF -> 1u
- C4: value 400u -> 470u; footprint Capacitor_SMD:CP_Elec_4x5.4 -> easyeda2kicad:CAP-TH_BD10.0-P5.00-D1.0-FD; moved to B.Cu
- C5: footprint Capacitor_SMD:C_0603_1608Metric -> Capacitor_SMD:C_0805_2012Metric
- C6, C7: value .1u -> 100n; footprint Capacitor_SMD:C_0603_1608Metric -> Capacitor_SMD:C_0402_1005Metric
- C9: value 0.1u -> 100n; footprint Capacitor_SMD:C_0603_1608Metric -> Capacitor_SMD:C_0402_1005Metric
- D1, D2, D3: value LED -> RED
- D10, D5, D6, D7, D9: value LED -> GREEN
- D4, D8: value LED -> YELLOW
- J1, J2: value Conn_01x03_Socket -> DS1023-1x3SF11; footprint Connector_PinHeader_2.54mm:PinHeader_1x03_P2.54mm_Vertical -> easyeda2kicad:HDR-TH_3P-P2.54-V-F-1; moved to B.Cu
- R1: value 1k -> 1K
- R12, R13, R14, R16, R18, R5: value R_Small_US -> 330
- R15: value R_Small_US -> 2.4k; footprint Resistor_SMD:R_0603_1608Metric -> Resistor_SMD:R_0805_2012Metric
- R2: value R_Small_US -> 10K
- R20: value 1k -> 1K; footprint Resistor_SMD:R_0603_1608Metric -> Resistor_SMD:R_0402_1005Metric
- R24, R25: footprint Resistor_SMD:R_0603_1608Metric -> Resistor_SMD:R_0805_2012Metric
- R3, R4: value R_Small_US -> 1K; footprint Resistor_SMD:R_0603_1608Metric -> Resistor_SMD:R_0402_1005Metric
- moved J1 149.4 mm to (76.6, 105.4), turned to 0 degrees
- moved Y1 145.6 mm to (87.1, 98.7), turned to 180 degrees
- moved R23 143.4 mm to (103.2, 111.5)
- moved C3 143.2 mm to (85.4, 102.2), turned to 0 degrees
- moved C9 143.1 mm to (101.4, 111.8)
- moved C12 141.5 mm to (83.2, 105.7), turned to 90 degrees
- moved C18 140.2 mm to (84.6, 105.7), turned to 90 degrees
- moved C2 140.1 mm to (88.9, 102.2), turned to 0 degrees
- moved C19 139.4 mm to (79.4, 111.5), turned to 180 degrees
- moved C10 139.2 mm to (79.5, 96.0)
- moved C11 139.2 mm to (79.5, 98.9)
- moved IC2 139.2 mm to (76.2, 97.4)
- moved R10 139.2 mm to (74.7, 93.9)
- moved R11 139.2 mm to (77.7, 93.4)
- moved R9 139.2 mm to (73.0, 98.7)
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Connections:
- D10 pad 2: /LED_EN+ -> /LED_EN_LED
- D8 pad 2: /LED_DO -> /LED_D_O
- R2 pad 1: Net-(D1-K) -> Net-(R2-Pad1)
- R2 pad 2: GND -> Net-(D1-K)
- R3 pad 2: GND -> Net-(R3-Pad2)
- R5 pad 2: GND -> Net-(R28-Pad2)
- U1 pad 11: /BTN_LED -> unconnected-(U1-GPIO8-Pad11)
- U1 pad 12: /BTN -> unconnected-(U1-GPIO9-Pad12)
- U1 pad 13: /ENC_A -> /ENC_B
- U1 pad 14: /ENC_B -> /ENC_A
- U1 pad 15: unconnected-(U1-GPIO12-Pad15) -> /LED_EN
- U1 pad 28: /LED_EN -> /LED_D
- U1 pad 36: unconnected-(U1-GPIO24-Pad36) -> /BOOT_LED
- U1 pad 37: /LED_D -> /P_SEN_LED
- U1 pad 38: unconnected-(U1-GPIO26_ADC0-Pad38) -> /P_SEN_O
- U1 pad 4: /P_SEN_O -> /LED_EN_LED
- U1 pad 5: /BOOT_LED -> /MGR_LED
- U1 pad 6: unconnected-(U1-GPIO4-Pad6) -> /ENC_LED
- U1 pad 7: unconnected-(U1-GPIO5-Pad7) -> /BTN_LED
- U1 pad 8: /ENC_LED -> /BTN
- U1 pad 9: /MGR_LED -> unconnected-(U1-GPIO7-Pad9)
Routing:
- net /LED_EN_LED: track 0.00 -> 23.6 mm
- net /MGR_LED: track 0.00 -> 23.0 mm
- net /ENC_LED: track 0.00 -> 22.3 mm
- net /BTN_LED: track 0.00 -> 21.7 mm
- net /BTN: track 34.0 -> 15.1 mm
- net /UART_RX: track 4.44 -> 21.5 mm
- net /ENC_A: track 28.7 -> 45.1 mm
- net Net-(SW1-A): track 23.2 -> 7.71 mm
- net GND: track 37.3 -> 52.0 mm, vias 43 -> 62
- net Net-(R23-Pad2): track 6.48 -> 18.3 mm
- net /ENC_B: track 24.4 -> 34.8 mm
- net /UART_TX: track 8.33 -> 18.4 mm
- net Net-(SW1-B): track 25.9 -> 16.7 mm
- net /SW_D: track 5.92 -> 14.0 mm, vias 0 -> 1
- net /QSPI_SD3: track 18.2 -> 10.3 mm
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Other:
- board size 80 x 40 mm -> 85 x 54 mm
- board text added: "24V"
- board text added: "3.3V"
- board text added: "5V"
- board text added: "Boot"
- board text added: "Btn"
- board text added: "CLK"
- board text added: "D"
- board text added: "Data"
- board text added: "Enc"
- board text added: "Fish Module 11/24 V0.1"
- board text added: "GND"
- board text added: "LED En"
- board text added: "Mgr"
- board text added: "P"
- board text added: "PSense"
- board text added: "RX"
- board text added: "SWD"
- board text added: "TX"

Commit message: Final version ready to roll
Parts:
- removed D12: D_Schottky, Diode_SMD:D_SMA
- removed D13: GREEN, LED_SMD:LED_0603_1608Metric
- removed J2: DS1023-1x3SF11, easyeda2kicad:HDR-TH_3P-P2.54-V-F-1
- removed R24, R25: 2.4k, Resistor_SMD:R_0805_2012Metric
- removed R26, R27: 330, Resistor_SMD:R_0603_1608Metric
- removed U3, U4: LTV357T-B, easyeda2kicad:SOP-4_L4.4-W4.0-P2.54-LS7.0-TL
- added Q2: FH38P03G6, easyeda2kicad:DFN-8_L3.3-W3.3-P0.65-BL-EP, F.Cu at (73.9, 95.4)
- CR1: footprint LD1117S33CTR:SOT-223_STM -> easyeda2kicad:SOT-223-4_L6.5-W3.5-P2.30-LS7.0-BR
- R17: value 330 -> 10k
- R19: value 100 -> 10k
- R20: value 1K -> 10k; footprint Resistor_SMD:R_0402_1005Metric -> Resistor_SMD:R_0603_1608Metric
- R21, R22, R23, R7: value 10K -> 10k
- moved R29 32.8 mm to (53.1, 119.9)
- moved R2 30.8 mm to (54.8, 119.9)
- moved D1 29.1 mm to (56.8, 119.9)
- moved R9 27.4 mm to (100.3, 97.2)
- moved R17 25.2 mm to (75.0, 102.2), turned to 0 degrees
- moved IC2 21.0 mm to (97.1, 95.5), turned to 0 degrees
- moved C11 20.5 mm to (99.2, 93.5)
- moved R10 19.5 mm to (93.9, 97.2), turned to 90 degrees
- moved R19 19.2 mm to (77.8, 96.0), turned to -90 degrees
- moved R20 17.3 mm to (80.2, 96.0), turned to 90 degrees
- moved Q1 16.8 mm to (78.8, 101.1), turned to -90 degrees
- moved C10 16.2 mm to (95.4, 92.9), turned to 90 degrees
- moved R11 13.6 mm to (91.2, 92.2), turned to 0 degrees
- moved D11 8.65 mm to (56.6, 113.7)
- moved D8 6.38 mm to (87.3, 90.9), turned to 90 degrees
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Connections:
- C4 pad 1: +24V -> Net-(C4-Pad1)
- J3 pad 1: +24V -> Net-(C4-Pad1)
- J3 pad 3: Net-(Q1-D) -> GND
- Q1 pad 1: Net-(Q1-G) -> /LED_EN
- R17 pad 1: Net-(R17-Pad1) -> GND
- R17 pad 2: GND -> /LED_EN
- R19 pad 1: Net-(Q1-G) -> Net-(Q2-G)
- R19 pad 2: Net-(R19-Pad2) -> +24V
- R20 pad 1: Net-(Q1-G) -> Net-(Q1-D)
- R20 pad 2: GND -> Net-(Q2-G)
- SW2 pad 1: /P_SEN -> +24V
- SW2 pad 3: +24V -> unconnected-(SW2-Pad3)
- U1 pad 15: /LED_EN -> /LED_D
- U1 pad 28: /LED_D -> /LED_EN
- U1 pad 37: /P_SEN_LED -> unconnected-(U1-GPIO25-Pad37)
- U1 pad 38: /P_SEN_O -> unconnected-(U1-GPIO26_ADC0-Pad38)
Routing:
- net +24V: track 0.00 -> 52.3 mm
- net /P_SEN_O: track 29.6 -> 0.00 mm, vias 2 -> 0
- net /P_SEN: track 23.4 -> 0.00 mm
- net Net-(C4-Pad1): track 0.00 -> 22.9 mm
- net /UART_RX: track 21.5 -> 0.00 mm
- net /UART_TX: track 18.4 -> 0.00 mm
- net +3.3V: track 16.9 -> 32.9 mm
- net /LED_D: track 13.1 -> 25.7 mm
- net Net-(Q1-D): track 12.6 -> 3.85 mm
- net /P_SEN_LED: track 7.33 -> 0.00 mm
- net Net-(D11-K): track 17.4 -> 12.1 mm
- net Net-(Q1-G): track 4.96 -> 0.00 mm
- net Net-(Q2-G): track 0.00 -> 4.93 mm
- net Net-(R24-Pad2): track 3.71 -> 0.00 mm
- net Net-(R26-Pad1): track 3.69 -> 0.00 mm
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- removed copper zone on F.Cu, net +24V
Other:
- board text added: "Fish Module 12/24 V0.3"
- board text removed: "Fish Module 11/24 V0.1"
- board text removed: "P"
- board text removed: "PSense"

Commit message: Finished lamp saving; cad v0.4
Parts:
- removed R1: 1K, Resistor_SMD:R_0402_1005Metric
- C2, C3: value 15p -> 12p
- Y1: value ABM8-272-T3 -> XYDBPCNANF-12MHZ; footprint ABM8-272-T3:ABM8272T3 -> easyeda2kicad:OSC-SMD_4P-L2.5-W2.0-BL
- moved C2 1.30 mm to (87.6, 102.2)
- turned Y1 to 0 degrees
Connections:
- C3 pad 2: Net-(Y1-CRYSTAL_2) -> /XOUT
- Y1 pad 1: /XIN -> /XOUT
- Y1 pad 3: Net-(Y1-CRYSTAL_2) -> /XIN
Routing:
- net /XOUT: track 3.21 -> 9.89 mm
- net Net-(Y1-CRYSTAL_2): track 5.66 -> 0.00 mm
- net /XIN: track 13.4 -> 12.5 mm
Other:
- board text added: "Fish Module 12/31 V0.4"
- board text removed: "Fish Module 12/24 V0.3"
